Commit message: changed import robot (paths for urdf/xml)

File: dodobot_v3/urdf/dodobot_v3.urdf (robot description, URDF)
Before this commit: robot dodobot_v3, 9 links, 8 joints
Links:
- link body_link: geometry collision mesh filename=../meshes/body_link.STL; visual mesh filename=../meshes/body_link.STL
- link left_link_1: geometry collision mesh filename=../meshes/left_link_1.STL; visual mesh filename=../meshes/left_link_1.STL
- link left_link_2: geometry collision mesh filename=../meshes/left_link_2.STL; visual mesh filename=../meshes/left_link_2.STL
- link left_link_3: geometry collision mesh filename=../meshes/left_link_3.STL; visual mesh filename=../meshes/left_link_3.STL
- link left_link_4: geometry collision mesh filename=../meshes/left_link_4.STL; visual mesh filename=../meshes/left_link_4.STL
- link right_link_1: geometry collision mesh filename=../meshes/right_link_1.STL; visual mesh filename=../meshes/right_link_1.STL
- link right_link_2: geometry collision mesh filename=../meshes/right_link_2.STL; visual mesh filename=../meshes/right_link_2.STL
- link right_link_3: geometry collision mesh filename=../meshes/right_link_3.STL; visual mesh filename=../meshes/right_link_3.STL
- link right_link_4: geometry collision mesh filename=../meshes/right_link_4.STL; visual mesh filename=../meshes/right_link_4.STL
