Commit message: path workaround finished. Now walking rewards has to be fixed

File: dodobot_v3/urdf/dodobot_v3_new.urdf (robot description, URDF)
Before this commit: robot dodobot_v3, 9 links, 8 joints
Links:
- link body_link: geometry collision box size=0.21 0.29 0.24; visual mesh filename=../meshes/body_link.STL
- link left_link_1: geometry collision capsule length=0.09 radius=0.026; visual mesh filename=../meshes/left_link_1.STL
- link left_link_2: geometry collision capsule length=0.185 radius=0.03; visual mesh filename=../meshes/left_link_2.STL
- link left_link_3: geometry collision capsule length=0.175 radius=0.03; visual mesh filename=../meshes/left_link_3.STL
- link left_link_4: geometry collision box size=0.06 0.095 0.034; visual mesh filename=../meshes/left_link_4.STL
- link right_link_1: geometry collision capsule length=0.09 radius=0.026; visual mesh filename=../meshes/right_link_1.STL
- link right_link_2: geometry collision capsule length=0.18 radius=0.03; visual mesh filename=../meshes/right_link_2.STL
- link right_link_3: geometry collision capsule length=0.175 radius=0.03; visual mesh filename=../meshes/right_link_3.STL
- link right_link_4: geometry collision box size=0.06 0.095 0.034; visual mesh filename=../meshes/right_link_4.STL

Commit message: Change upper limit of joint from -1.5 to 1.5 of left_joint_2

File: dodobot_v3/urdf/dodobot_v3_new.urdf (robot description, URDF)
Before this commit: robot dodobot_v3, 9 links, 8 joints
Joints:
- joint left_joint_2: limit lower=-1.5 upper=-1.5 effort=3 velocity=5 -> lower=-1.5 upper=1.5 effort=3 velocity=5

Commit message: Refactor URDF: Simplify collision and align joints
Updated collision geometry to use primitive shapes, removed mimic joints, and corrected joint axis alignments.

File: dodobot_v3/urdf/dodobot_v3_new.urdf (robot description, URDF)
Before this commit: robot dodobot_v3, 9 links, 8 joints
Links:
- added link base_link
- link body_link: geometry collision box size=0.21 0.29 0.23; visual mesh filename=package://dodobot_v3/meshes/body_link.STL
- link left_link_1: geometry visual mesh filename=package://dodobot_v3/meshes/left_link_1.STL
- link left_link_2: geometry collision capsule length=0.18 radius=0.03; visual mesh filename=package://dodobot_v3/meshes/left_link_2.STL
- link left_link_3: geometry collision capsule length=0.14 radius=0.03; visual mesh filename=package://dodobot_v3/meshes/left_link_3.STL
- link left_link_4: geometry collision box size=0.095 0.036 0.0615; visual mesh filename=package://dodobot_v3/meshes/left_link_4.STL
- link right_link_1: geometry visual mesh filename=package://dodobot_v3/meshes/right_link_1.STL
- link right_link_3: geometry collision capsule length=0.14 radius=0.03; visual mesh filename=package://dodobot_v3/meshes/right_link_3.STL
- link right_link_4: geometry collision box size=0.095 0.036 0.0615; visual mesh filename=package://dodobot_v3/meshes/right_link_4.STL
Joints:
- added joint base_to_body: type fixed, parent base_link, child body_link, origin xyz=0 0 0 rpy=0 0 -1.5708
- joint left_joint_1: axis 0 0 1 -> -1 0 0; origin xyz=-0.066 0 -0.092 rpy=1.5708 0 3.1416 -> xyz=-0.066 0 -0.092 rpy=0 0 1.5708
- joint left_joint_2: axis 0 0 1 -> 0 -1 0; origin xyz=0.01295 -0.04009 -0.01705 rpy=1.5708 0 -1.5708 -> xyz=-0.01705 0.01295 -0.04009 rpy=0 0 0
- joint left_joint_3: axis 0 0 1 -> 0 -1 0; origin xyz=0.2 0 -0.03745 rpy=0 0 0 -> xyz=0 0.03745 -0.2 rpy=0 0 0
- joint left_joint_4: axis 0 0 1 -> 0 -1 0; origin xyz=0.2 0 -0.03745 rpy=0 0 0 -> xyz=0 0.03745 -0.2 rpy=0 0 0
- joint right_joint_1: axis 0 0 -1 -> -1 0 0; origin xyz=0.066 0 -0.092 rpy=1.5708 0 3.1416 -> xyz=0.066 0 -0.092 rpy=0 0 1.5708
- joint right_joint_2: axis 0 0 1 -> 0 -1 0; origin xyz=0 -0.04009 -0.01705 rpy=1.5708 0 -1.5708 -> xyz=-0.01705 0 -0.04009 rpy=0 0 0
- joint right_joint_3: axis 0 0 1 -> 0 -1 0; origin xyz=0.2 0 0.0504 rpy=0 0 0 -> xyz=0 -0.0504 -0.2 rpy=0 0 0
- joint right_joint_4: axis 0 0 1 -> 0 -1 0; origin xyz=0.2 0 0.03745 rpy=0 0 0 -> xyz=0 -0.03745 -0.2 rpy=0 0 0
